Commit message: Added laser scanner

File: src/myrobot_description/urdf/myrobot.gazebo.xacro (robot description, xacro)
@@ -69,3 +69,38 @@
         <xacro:set_link_friction link="ballcaster" friction="0"/>
     </xacro:macro>
+     <gazebo reference="laser_link">
+    <sensor type="ray" name="head_hokuyo_sensor">
+      <pose>0 0 0 0 0 0</pose>
+      <visualize>true</visualize>
+      <update_rate>10</update_rate>
+      <ray>
+        <scan>
+          <horizontal>
+            <samples>360</samples>
+            <resolution>1</resolution>
+            <min_angle>-1.570796</min_angle>
+            <max_angle>1.570796</max_angle>
+          </horizontal>
+        </scan>
+        <range>
+          <min>0.14</min>
+          <max>30.0</max>
+          <resolution>0.01</resolution>
+        </range>
+        <noise>
+          <type>gaussian</type>
+          <!-- Noise parameters based on published spec for Hokuyo laser
+               achieving "+-30mm" accuracy at range < 10m.  A mean of 0.0m and
+               stddev of 0.01m will put 99.7% of samples within 0.03m of the true
+               reading. -->
+          <mean>0.0</mean>
+          <stddev>0.01</stddev>
+        </noise>
+      </ray>
+      <plugin name="gazebo_ros_head_hokuyo_controller" filename="libgazebo_ros_laser.so">
+        <topicName>scan</topicName>
+        <frameName>laser_link</frameName>
+      </plugin>
+    </sensor>
+  </gazebo>
 </robot>

File: src/myrobot_description/urdf/myrobot.urdf.xacro (robot description, xacro)
@@ -84,4 +84,13 @@
         <xacro:cylinder_inertia m="${wheel_mass}" r="${wheel_r}" l="${wheel_w}"/>
     </link>
+    <!-- ===== SENSORS ===== -->
+    <link name="laser_link">
+        <visual>
+            <origin xyz="0.0 0.0 -0.025"/>
+            <geometry>
+                <cylinder radius="0.02" length="0.03"/>
+            </geometry>
+        </visual>
+    </link>
     <!-- ===== JOINTS ===== -->
     <joint name="base_chasis" type="fixed">
@@ -109,4 +118,9 @@
         <limit effort="100" velocity="100.0"/>
     </joint>
+    <joint name="base_laser" type="fixed">
+        <origin xyz="${pos_x_joint} 0 0.10"/>
+        <parent link="chassis"/>
+        <child link="laser_link"/>
+    </joint>
     <!-- ===== GAZEBO ===== -->
     <xacro:set_diff_drive base_width="${base_width}" wheel_width="${wheel_w}" wheel_radius="${wheel_r}"/>

Commit message: Added laser

File: src/myrobot_description/urdf/myrobot.gazebo.xacro (robot description, xacro)
@@ -73,17 +73,17 @@
       <pose>0 0 0 0 0 0</pose>
       <visualize>true</visualize>
-      <update_rate>10</update_rate>
+      <update_rate>40</update_rate>
       <ray>
         <scan>
           <horizontal>
-            <samples>360</samples>
+            <samples>720</samples>
             <resolution>1</resolution>
-            <min_angle>-1.570796</min_angle>
-            <max_angle>1.570796</max_angle>
+            <min_angle>-3.14159265</min_angle>
+            <max_angle>3.14159265</max_angle>
           </horizontal>
         </scan>
         <range>
-          <min>0.14</min>
-          <max>30.0</max>
+          <min>0.2</min>
+          <max>12.0</max>
           <resolution>0.01</resolution>
         </range>
@@ -98,5 +98,5 @@
         </noise>
       </ray>
-      <plugin name="gazebo_ros_head_hokuyo_controller" filename="libgazebo_ros_laser.so">
+      <plugin name="gazebo_ros_head_rplidar_controller" filename="libgazebo_ros_laser.so">
         <topicName>scan</topicName>
         <frameName>laser_link</frameName>

File: src/myrobot_description/urdf/myrobot.urdf.xacro (robot description, xacro)
@@ -87,7 +87,7 @@
     <link name="laser_link">
         <visual>
-            <origin xyz="0.0 0.0 -0.025"/>
+            <origin xyz="0.0 0.0 0" rpy="0 0 3.14"/>
             <geometry>
-                <cylinder radius="0.02" length="0.03"/>
+                <mesh filename="file://$(find myrobot_description)/meshes/rplidar-a2.stl"/>
             </geometry>
         </visual>
@@ -119,5 +119,5 @@
     </joint>
     <joint name="base_laser" type="fixed">
-        <origin xyz="${pos_x_joint} 0 0.10"/>
+        <origin xyz="${pos_x_joint} 0 ${base_height/2 + 0.028}" rpy="0 0 ${3.14}"/>
         <parent link="chassis"/>
         <child link="laser_link"/>

Commit message: Added laserv2

File: src/myrobot_description/urdf/myrobot.gazebo.xacro (robot description, xacro)
@@ -55,4 +55,7 @@
         <material>Gazebo/Purple </material>
     </gazebo>
+    <gazebo reference="laser_link">
+        <material>Gazebo/Black </material>
+    </gazebo>
     <xacro:macro name="set_link_friction" params="link friction">
         <gazebo reference="${link}">
@@ -70,5 +73,5 @@
     </xacro:macro>
      <gazebo reference="laser_link">
-    <sensor type="ray" name="head_hokuyo_sensor">
+    <sensor type="ray" name="head_rplidar_sensor">
       <pose>0 0 0 0 0 0</pose>
       <visualize>true</visualize>
